Commit message: Added Gazebo functionality

File: description/robot_core.xacro (robot description, xacro)
@@ -17,4 +17,6 @@
             <geometry>
                 <box size="0.66 0.548 0.281" />
+                <!-- importing the mesh didn't work... -->
+                <!-- mesh filename="package://bunker_mini/description/bunker_mini.stl" /-->
             </geometry>
             <material name="white" />
@@ -26,5 +28,11 @@
             </geometry>
         </collision>
+        <xacro:inertial_box mass="2" x="0.66" y="0.548" z="0.281">
+            <origin xyz="0.33 0 0.1405" rpy="0 0 0" />
+        </xacro:inertial_box>
     </link>
+    <gazebo reference="chassis">
+        <material>Gazebo/White</material>
+    </gazebo>
     <!-- LEFT WHEEL LINK -->
     <joint name="left_wheel_joint" type="continuous">
@@ -49,5 +57,11 @@
             </geometry>
         </collision>
+        <xacro:inertial_cylinder mass="0.1" length="0.04" radius="0.05">
+            <origin xyz="0 0 0 " rpy="0 0 0" />
+        </xacro:inertial_cylinder>
     </link>
+    <gazebo reference="left_wheel">
+        <material>Gazebo/Blue</material>
+    </gazebo>
     <!-- RIGHT WHEEL LINK -->
     <joint name="right_wheel_joint" type="continuous">
@@ -72,5 +86,11 @@
             </geometry>
         </collision>
+        <xacro:inertial_cylinder mass="0.1" length="0.04" radius="0.05">
+            <origin xyz="0 0 0 " rpy="0 0 0" />
+        </xacro:inertial_cylinder>
     </link>
+    <gazebo reference="right_wheel">
+        <material>Gazebo/Blue</material>
+    </gazebo>
     <!-- FRONT CASTER WHEEL LINK -->
     <joint name="front_caster_wheel_joint" type="fixed">
@@ -91,5 +111,13 @@
             </geometry>
         </collision>
+        <xacro:inertial_sphere mass="0.1" radius="0.05">
+            <origin xyz="0 0 0" rpy="0 0 0" />
+        </xacro:inertial_sphere>
     </link>
+    <gazebo reference="front_caster_wheel">
+        <material>Gazebo/Black</material>
+        <mu1 value="0.001" />
+        <mu2 value="0.001" />
+    </gazebo>
     <!-- REAR CASTER WHEEL LINK -->
     <joint name="rear_caster_wheel_joint" type="fixed">
@@ -110,4 +138,12 @@
             </geometry>
         </collision>
+        <xacro:inertial_sphere mass="0.1" radius="0.05">
+            <origin xyz="0 0 0" rpy="0 0 0" />
+        </xacro:inertial_sphere>
     </link>
+    <gazebo reference="rear_caster_wheel">
+        <material>Gazebo/Black</material>
+        <mu1 value="0.001" />
+        <mu2 value="0.001" />
+    </gazebo>
 </robot>
