Commit message: Update lnd712.xacro
Changed colour and geometry

File: description/lnd712.xacro (robot description, xacro)
@@ -10,7 +10,7 @@
         <visual>
             <geometry>
-                <cylinder radius="0.038" length="0.041" />
+                <cylinder radius="0.0151" length="0.0492" />
             </geometry>
-            <material name="red" />
+            <material name="orange" />
         </visual>
         <collision>
